Commit message: Updating rosbee_model

File: rosbee_ros/rosbee_description/urdf/components/kinect.urdf.xacro (robot description, xacro)
@@ -48,4 +48,5 @@
         <origin xyz="0 0 0" rpy="0 0 0"/>
         <geometry>
+          <!--<box size="${kinect_length} ${kinect_width} ${kinect_height}"/>-->
           <mesh filename="package://rosbee_description/meshes/kinect.stl" scale="0.001 0.001 0.001"/>
         </geometry>
