Commit message: Cleaned up file names

File: rosbee_ros/rosbee_description/urdf/components/motor_wheel_unit.urdf.xacro (robot description, xacro)
@@ -27,5 +27,5 @@
       <visual>
       	<geometry>
-      		<mesh filename="package://rosbee_description/meshes/500093_RVS_motorsteun_rosbee.stl" scale="0.02541 0.02541 0.02541"/>
+      		<mesh filename="package://rosbee_description/meshes/500093_rvs_motormount_.stl" scale="0.02541 0.02541 0.02541"/>
       	</geometry>
       	<origin rpy="0 ${-M_PI/2} ${-reflect * M_PI/2}" xyz="0 ${reflect * motor_mount_vis_offset_y} 0"/>
@@ -43,8 +43,6 @@
       <visual>
       <geometry>
-        <!--<cylinder length="${motor_height}" radius="${motor_radius}"/>-->
-        <mesh filename="package://rosbee_description/meshes/1443_metal_gearmotor2.stl" scale="0.001 0.001 0.001"/>
+        <mesh filename="package://rosbee_description/meshes/1443_metal_gearmotor.stl" scale="0.001 0.001 0.001"/>
       </geometry>
-      <!--<origin rpy="0 0 0" xyz="0 -0.003 0.007"/>-->
   		<origin rpy="0 0 ${(M_PI/2)+(reflect * (M_PI/2))}" xyz="0 ${reflect*0.003} 0.007"/>
       <material name="black">
@@ -66,5 +64,5 @@
       <visual>
       <geometry>
-        <mesh filename="package://rosbee_description/meshes/wheel_hub.stl" scale="0.001 0.001 0.001"/>
+        <mesh filename="package://rosbee_description/meshes/bane_bots_wheel_hub.stl" scale="0.001 0.001 0.001"/>
       </geometry>
       <origin rpy="0 0 0" xyz="0 0 0"/>
@@ -77,5 +75,5 @@
       <visual>
       <geometry>
-        <mesh filename="package://rosbee_description/meshes/tire.stl" scale="0.001 0.001 0.001"/>
+        <mesh filename="package://rosbee_description/meshes/bane_bots_tire.stl" scale="0.001 0.001 0.001"/>
       </geometry>
       <origin rpy="0 0 0" xyz="0 0 0"/>

File: rosbee_ros/rosbee_description/urdf/components/swivel_wheel_unit.urdf.xacro (robot description, xacro)
@@ -1,8 +1,5 @@
 <?xml version="1.0"?>
 <robot xmlns:xacro="http://www.ros.org/wiki/xacro" name="rosbee">
-  <!-- motor_wheel_unit properties -->
-  <property name="swivel_mount_width" value="0.057" />
-  <property name="swivel_mount_length" value="0.057" />
-  <property name="swivel_mount_height" value="0.0065" />
+  <!-- swivel wheel unit properties -->
   <property name="swivel_bracket_offset_z" value="-0.007" />
   <property name="swivel_wheel_offset_z" value="-0.055" />
