Commit message: Updating model files

File: rosbee_ros/rosbee_description/robots/rosbee.urdf.xacro (robot description, xacro)
@@ -1,39 +1,42 @@
 <?xml version="1.0"?>
-<robot xmlns:sensor="http://playerstage.sourceforge.net/gazebo/xmlschema/#sensor"
-       xmlns:controller="http://playerstage.sourceforge.net/gazebo/xmlschema/#controller"
-       xmlns:interface="http://playerstage.sourceforge.net/gazebo/xmlschema/#interface"
-       xmlns:xacro="http://playerstage.sourceforge.net/gazebo/xmlschema/#interface"
-       name="rosbee2a" >
+<robot xmlns:xacro="http://www.ros.org/wiki/xacro" name="rosbee">
   <!-- Rosbee Frame -->
-  <xacro:include filename="$(find rosbee_description)/urdf/top_plate.urdf.xacro" />
-  <xacro:include filename="$(find rosbee_description)/urdf/bottom_plate.urdf.xacro" />
-  <xacro:include filename="$(find rosbee_description)/urdf/spacer.urdf.xacro" />
-  <!-- Rosbee 2a kinect -->
-  <!--
-  <xacro:include filename="$(find rosbee_description)/urdf/sensors/kinect/kinect.urdf.xacro" />
-  -->
+  <xacro:include filename="$(find rosbee_description)/urdf/components/top_plate.urdf.xacro" />
+  <xacro:include filename="$(find rosbee_description)/urdf/components/bottom_plate.urdf.xacro" />
+  <xacro:include filename="$(find rosbee_description)/urdf/components/spacer.urdf.xacro" />
+  <xacro:include filename="$(find rosbee_description)/urdf/components/kinect.urdf.xacro" />
+  <link name="base_link">
+    <visual>
+        <!--<origin xyz="0 0 0" rpy="0 0 0" />-->
+      <geometry>
+        <box size="0.01 0.01 0.01" />
+      </geometry>
+    </visual>
+  </link>
+  <joint name="base_link_joint" type="fixed">
+     <origin xyz="0 0 0" rpy="0 0 0" />
+     <child link="bottom_plate_link" />
+     <parent link="base_link"/>
+  </joint>
   <xacro:bottom_plate name="bottom_plate" parent="base">
     <origin xyz="0 0 0.104" rpy="0 0 0" />
   </xacro:bottom_plate>
   <xacro:spacer name="spacer_1" parent="bottom_plate">
-    <origin xyz="0 0 0.067" rpy="0 0 0" />
+    <origin xyz="0.105 0.105 0.000" rpy="0 0 0" />
   </xacro:spacer>
   <xacro:spacer name="spacer_2" parent="bottom_plate">
-    <origin xyz="0 0 0.067" rpy="0 0 0" />
+    <origin xyz="0.105 -0.105 0.000" rpy="0 0 0" />
   </xacro:spacer>
   <xacro:spacer name="spacer_3" parent="bottom_plate">
-    <origin xyz="0 0 0.067" rpy="0 0 0" />
+    <origin xyz="-0.105 -0.105 0.000" rpy="0 0 0" />
   </xacro:spacer>
   <xacro:spacer name="spacer_4" parent="bottom_plate">
-    <origin xyz="0 0 0.067" rpy="0 0 0" />
+    <origin xyz="-0.105 0.105 0.000" rpy="0 0 0" />
   </xacro:spacer>
   <xacro:top_plate name="top_plate" parent="bottom_plate">
     <origin xyz="0 0 0.067" rpy="0 0 0" />
-  </xacro:bottom_plate>
-  <!--
-  <xacro:sensor_kinect parent="pan_tilt_yaw_link">
-    <origin xyz="-0.0000 -0.0000 0.0287" rpy="0 0 0"/>
-    <!-- <origin xyz="-0.0011 -0.0003 0.03" rpy="0 0 0"/> -->
+  </xacro:top_plate>
+  <xacro:sensor_kinect parent="bottom_plate_link">
+    <origin xyz="0.0675 0.0000 0.032" rpy="0 0 0"/>
   </xacro:sensor_kinect>
-  -->
 </robot>

File: rosbee_ros/rosbee_description/urdf/components/bottom_plate.urdf.xacro (robot description, xacro)
@@ -1,10 +1,7 @@
 <?xml version="1.0"?>
-<robot xmlns:sensor="http://playerstage.sourceforge.net/gazebo/xmlschema/#sensor"
-       xmlns:controller="http://playerstage.sourceforge.net/gazebo/xmlschema/#controller"
-       xmlns:interface="http://playerstage.sourceforge.net/gazebo/xmlschema/#interface"
-       xmlns:xacro="http://ros.org/wiki/xacro">
+<robot xmlns:xacro="http://www.ros.org/wiki/xacro" name="rosbee">
   <!-- bottom_plate properties -->
-  <property name="diameter" value="0.390" />
-  <property name="height" value="0.008" />
+  <property name="bottom_diameter" value="0.390" />
+  <property name="bottom_height" value="0.008" />
   <xacro:macro name="bottom_plate" params="name parent *origin">
     <joint name="${name}_joint" type="fixed">
@@ -16,9 +13,9 @@
       <visual>
       <geometry>
-        <cylinder radius="${radius}" length="${height}" />
+        <cylinder radius="${bottom_diameter/2}" length="${bottom_height}" />
       </geometry>
       <origin rpy="0 0 0" xyz="0 0 0"/>
       <material name="black">
-        <color rgba="0.000 0.000 0.000 1"/>
+        <color rgba="0.1 0.1 0.1 1"/>
       </material>
     </visual>

File: rosbee_ros/rosbee_description/urdf/components/kinect.urdf.xacro (robot description, xacro)
@@ -26,5 +26,5 @@
     </link>
     <joint name="camera_rgb_optical_joint" type="fixed">
-      <origin xyz="0 0 0" rpy="${M_PI/2} 0 0" />
+      <origin xyz="0 0 0" rpy="${M_PI/2} 0 ${-M_PI/2}" />
       <parent link="camera_rgb_frame" />
       <child link="camera_rgb_optical_frame" />
@@ -46,5 +46,5 @@
     <link name="camera_link">
       <visual>
-        <origin xyz="0 0 0" rpy="0 0 0"/>
+        <origin xyz="0 0 0" rpy="0 0 ${-M_PI}"/>
         <geometry>
           <!--<box size="${kinect_length} ${kinect_width} ${kinect_height}"/>-->

File: rosbee_ros/rosbee_description/urdf/components/spacer.urdf.xacro (robot description, xacro)
@@ -1,10 +1,7 @@
 <?xml version="1.0"?>
-<robot xmlns:sensor="http://playerstage.sourceforge.net/gazebo/xmlschema/#sensor"
-       xmlns:controller="http://playerstage.sourceforge.net/gazebo/xmlschema/#controller"
-       xmlns:interface="http://playerstage.sourceforge.net/gazebo/xmlschema/#interface"
-       xmlns:xacro="http://ros.org/wiki/xacro">
+<robot xmlns:xacro="http://www.ros.org/wiki/xacro" name="rosbee">
   <!-- spacer properties -->
-  <property name="diameter" value="0.015" />
-  <property name="height" value="0.059" />
+  <property name="spacer_diameter" value="0.015" />
+  <property name="spacer_height" value="0.059" />
   <xacro:macro name="spacer" params="name parent *origin">
     <joint name="${name}_joint" type="fixed">
@@ -16,9 +13,9 @@
       <visual>
       <geometry>
-        <cylinder radius="${radius}" length="${height}" />
+        <cylinder radius="${spacer_diameter/2.000}" length="${spacer_height}" />
       </geometry>
-      <origin rpy="0 0 0" xyz="0 0 0"/>
+      <origin rpy="0 0 0" xyz="0 0 ${(spacer_height / 2.000) + 0.004}"/>
       <material name="black">
-        <color rgba="0.000 0.000 0.000 1"/>
+        <color rgba="0.1 0.1 0.1 1"/>
       </material>
     </visual>

File: rosbee_ros/rosbee_description/urdf/components/top_plate.urdf.xacro (robot description, xacro)
@@ -1,7 +1,4 @@
 <?xml version="1.0"?>
-<robot xmlns:sensor="http://playerstage.sourceforge.net/gazebo/xmlschema/#sensor"
-       xmlns:controller="http://playerstage.sourceforge.net/gazebo/xmlschema/#controller"
-       xmlns:interface="http://playerstage.sourceforge.net/gazebo/xmlschema/#interface"
-       xmlns:xacro="http://ros.org/wiki/xacro">
+<robot xmlns:xacro="http://www.ros.org/wiki/xacro" name="rosbee">
   <!-- top_plate properties -->
   <property name="top_plate_width" value="0.250" />
@@ -21,7 +18,7 @@
       <origin rpy="0 0 0" xyz="0 0 0"/>
       <material name="black">
-        <color rgba="0.000 0.000 0.000 1"/>
+        <color rgba="0.1 0.1 0.1 1"/>
       </material>
-    </visual>
+      </visual>
     </link>
   </xacro:macro>

Commit message: bottom_plate_link renamed to base_link

File: rosbee_ros/rosbee_description/robots/rosbee.urdf.xacro (robot description, xacro)
@@ -1,41 +1,43 @@
 <?xml version="1.0"?>
 <robot xmlns:xacro="http://www.ros.org/wiki/xacro" name="rosbee">
-  <!-- Rosbee Frame -->
+  <!--  Includes for various component xacros -->
   <xacro:include filename="$(find rosbee_description)/urdf/components/top_plate.urdf.xacro" />
   <xacro:include filename="$(find rosbee_description)/urdf/components/bottom_plate.urdf.xacro" />
   <xacro:include filename="$(find rosbee_description)/urdf/components/spacer.urdf.xacro" />
   <xacro:include filename="$(find rosbee_description)/urdf/components/kinect.urdf.xacro" />
-  <link name="base_link">
-    <visual>
-        <!--<origin xyz="0 0 0" rpy="0 0 0" />-->
-      <geometry>
-        <box size="0.01 0.01 0.01" />
-      </geometry>
-    </visual>
-  </link>
+  <!--
+        base_footprint is a fictitious link(frame)
+        that is on the ground right below base_link origin,
+        navigation stack dedpends on this frame
+  -->
+  <link name="base_footprint_link"></link>
   <joint name="base_link_joint" type="fixed">
-     <origin xyz="0 0 0" rpy="0 0 0" />
-     <child link="bottom_plate_link" />
-     <parent link="base_link"/>
+     <origin xyz="0 0 0.104" rpy="0 0 0" />
+     <child link="base_link" />
+     <parent link="base_footprint_link"/>
   </joint>
-  <xacro:bottom_plate name="bottom_plate" parent="base">
+  <!-- The bottom plate acts as our base_link -->
+  <xacro:bottom_plate name="base" parent="base_footprint">
     <origin xyz="0 0 0.104" rpy="0 0 0" />
   </xacro:bottom_plate>
-  <xacro:spacer name="spacer_1" parent="bottom_plate">
+  <!--  Spacers between bottom_plate and top_plate -->
+  <xacro:spacer name="spacer_1" parent="base">
     <origin xyz="0.105 0.105 0.000" rpy="0 0 0" />
   </xacro:spacer>
-  <xacro:spacer name="spacer_2" parent="bottom_plate">
+  <xacro:spacer name="spacer_2" parent="base">
     <origin xyz="0.105 -0.105 0.000" rpy="0 0 0" />
   </xacro:spacer>
-  <xacro:spacer name="spacer_3" parent="bottom_plate">
+  <xacro:spacer name="spacer_3" parent="base">
     <origin xyz="-0.105 -0.105 0.000" rpy="0 0 0" />
   </xacro:spacer>
-  <xacro:spacer name="spacer_4" parent="bottom_plate">
+  <xacro:spacer name="spacer_4" parent="base">
     <origin xyz="-0.105 0.105 0.000" rpy="0 0 0" />
   </xacro:spacer>
-  <xacro:top_plate name="top_plate" parent="bottom_plate">
+  <xacro:top_plate name="top_plate" parent="base">
     <origin xyz="0 0 0.067" rpy="0 0 0" />
   </xacro:top_plate>
-  <xacro:sensor_kinect parent="bottom_plate_link">
+  <!-- TODO add wheel units -->
+  <!--  kinect sensor -->
+  <xacro:sensor_kinect parent="base_link">
     <origin xyz="0.0675 0.0000 0.032" rpy="0 0 0"/>
   </xacro:sensor_kinect>

Commit message: First complete model

File: rosbee_ros/rosbee_description/robots/rosbee.urdf.xacro (robot description, xacro)
@@ -6,39 +6,54 @@
   <xacro:include filename="$(find rosbee_description)/urdf/components/spacer.urdf.xacro" />
   <xacro:include filename="$(find rosbee_description)/urdf/components/kinect.urdf.xacro" />
-  <!--
-        base_footprint is a fictitious link(frame)
-        that is on the ground right below base_link origin,
-        navigation stack dedpends on this frame
-  -->
-  <link name="base_footprint_link"></link>
-  <joint name="base_link_joint" type="fixed">
-     <origin xyz="0 0 0.104" rpy="0 0 0" />
-     <child link="base_link" />
-     <parent link="base_footprint_link"/>
-  </joint>
+  <xacro:include filename="$(find rosbee_description)/urdf/components/motor_wheel_unit.urdf.xacro" />
+  <xacro:include filename="$(find rosbee_description)/urdf/components/swivel_wheel_unit.urdf.xacro" />
   <!-- The bottom plate acts as our base_link -->
-  <xacro:bottom_plate name="base" parent="base_footprint">
+  <xacro:bottom_plate name="base">
     <origin xyz="0 0 0.104" rpy="0 0 0" />
   </xacro:bottom_plate>
   <!--  Spacers between bottom_plate and top_plate -->
   <xacro:spacer name="spacer_1" parent="base">
-    <origin xyz="0.105 0.105 0.000" rpy="0 0 0" />
+    <origin xyz="0.10 0.10 0.000" rpy="0 0 0" />
   </xacro:spacer>
   <xacro:spacer name="spacer_2" parent="base">
-    <origin xyz="0.105 -0.105 0.000" rpy="0 0 0" />
+    <origin xyz="0.10 -0.10 0.000" rpy="0 0 0" />
   </xacro:spacer>
   <xacro:spacer name="spacer_3" parent="base">
-    <origin xyz="-0.105 -0.105 0.000" rpy="0 0 0" />
+    <origin xyz="-0.10 -0.10 0.000" rpy="0 0 0" />
   </xacro:spacer>
   <xacro:spacer name="spacer_4" parent="base">
-    <origin xyz="-0.105 0.105 0.000" rpy="0 0 0" />
+    <origin xyz="-0.10 0.10 0.000" rpy="0 0 0" />
   </xacro:spacer>
   <xacro:top_plate name="top_plate" parent="base">
-    <origin xyz="0 0 0.067" rpy="0 0 0" />
+    <origin xyz="0 0 0.059" rpy="0 0 0" />
   </xacro:top_plate>
   <!-- TODO add wheel units -->
+  <xacro:motor_wheel_unit name="left"
+                          parent="base"
+                          reflect="1"
+                          offset_x="0"
+                          offset_y="0.1225"
+                          offset_z="-0.003"/>
+  <xacro:motor_wheel_unit name="right"
+                          parent="base"
+                          reflect="-1"
+                          offset_x="0"
+                          offset_y="0.1225"
+                          offset_z="-0.003"/>
+  <xacro:swivel_wheel_unit name="front"
+                          parent="base"
+                          reflect="1"
+                          offset_x="0.135"
+                          offset_y="0"
+                          offset_z="-0.0050"/>
+  <xacro:swivel_wheel_unit name="rear"
+                          parent="base"
+                          reflect="-1"
+                          offset_x="0.135"
+                          offset_y="0"
+                          offset_z="-0.0050"/>
   <!--  kinect sensor -->
-  <xacro:sensor_kinect parent="base_link">
-    <origin xyz="0.0675 0.0000 0.032" rpy="0 0 0"/>
+  <xacro:sensor_kinect parent="top_plate_link">
+    <origin xyz="-0.100 0.0000 0.126" rpy="0 0 -0.018516402"/>
   </xacro:sensor_kinect>
 </robot>

File: rosbee_ros/rosbee_description/urdf/components/bottom_plate.urdf.xacro (robot description, xacro)
@@ -4,16 +4,12 @@
   <property name="bottom_diameter" value="0.390" />
   <property name="bottom_height" value="0.008" />
-  <xacro:macro name="bottom_plate" params="name parent *origin">
-    <joint name="${name}_joint" type="fixed">
-      <insert_block name="origin" />
-      <parent link="${parent}_link"/>
-      <child link="${name}_link"/>
-    </joint>
+  <property name="bottom_plate_offset_z" value="0.005" />
+  <xacro:macro name="bottom_plate" params="name *origin">
     <link name="${name}_link">
       <visual>
       <geometry>
-        <cylinder radius="${bottom_diameter/2}" length="${bottom_height}" />
+        <mesh filename="package://rosbee_description/meshes/500068B_rosbee_base_plate_350.stl" scale="0.001 0.001 0.001"/>
       </geometry>
-      <origin rpy="0 0 0" xyz="0 0 0"/>
+      <origin rpy="0 0 0" xyz="0 0 ${bottom_plate_offset_z}"/>
       <material name="black">
         <color rgba="0.1 0.1 0.1 1"/>
@@ -21,4 +17,15 @@
     </visual>
     </link>
+    <!--
+        base_footprint is a fictitious link(frame)
+        that is on the ground right below base_link origin,
+        navigation stack dedpends on this frame
+    -->
+    <link name="base_footprint"/>
+    <joint name="${name}_footprint_joint" type="fixed">
+      <insert_block name="origin" />
+      <child link="${name}_link"/>
+      <parent link="${name}_footprint"/>
+    </joint>
   </xacro:macro>
 </robot>

File: rosbee_ros/rosbee_description/urdf/components/motor_wheel_unit.urdf.xacro (robot description, xacro)
@@ -1 +1,88 @@
-<!-- xacro for wheel units -->
+<?xml version="1.0"?>
+<robot xmlns:xacro="http://www.ros.org/wiki/xacro" name="rosbee">
+  <!-- motor_wheel_unit properties -->
+  <property name="motor_mount_width" value="0.055" />
+  <property name="motor_mount_length" value="0.055" />
+  <property name="motor_mount_height" value="0.055" />
+  <property name="motor_mount_vis_offset_y" value="0.0275" />
+  <property name="motor_radius" value="0.017" />
+  <property name="motor_height" value="0.083" />
+  <property name="motor_trans_z" value="-0.0402" />
+	<property name="wheel_gap" value="0.005" />
+  <property name="wheel_radius" value="0.062" />
+  <property name="wheel_height" value="0.019" />
+  <property name="wheel_trans_y" value="0.019" />
+  <xacro:macro name="motor_wheel_unit" params="	name
+  																							parent
+  																							reflect
+  																							offset_x
+  																							offset_y
+  																							offset_z">
+    <joint name="${name}_motor_mount_joint" type="fixed">
+      <origin xyz="${offset_x} ${reflect * offset_y} ${offset_z}" rpy="0 0 0" />
+      <parent link="${parent}_link"/>
+      <child link="${name}_motor_mount_link"/>
+    </joint>
+    <link name="${name}_motor_mount_link">
+      <visual>
+      	<geometry>
+      		<mesh filename="package://rosbee_description/meshes/500093_RVS_motorsteun_rosbee.stl" scale="0.02541 0.02541 0.02541"/>
+      	</geometry>
+      	<origin rpy="0 ${-M_PI/2} ${-reflect * M_PI/2}" xyz="0 ${reflect * motor_mount_vis_offset_y} 0"/>
+      	<material name="black">
+        	<color rgba="0.1 0.1 0.1 1"/>
+      	</material>
+      </visual>
+    </link>
+    <joint name="${name}_motor_joint" type="fixed">
+      <origin xyz="0 0 ${motor_trans_z}" rpy="0 0 0" />
+      <parent link="${name}_motor_mount_link"/>
+      <child link="${name}_motor_link"/>
+    </joint>
+    <link name="${name}_motor_link">
+      <visual>
+      <geometry>
+        <!--<cylinder length="${motor_height}" radius="${motor_radius}"/>-->
+        <mesh filename="package://rosbee_description/meshes/1443_metal_gearmotor2.stl" scale="0.001 0.001 0.001"/>
+      </geometry>
+      <!--<origin rpy="0 0 0" xyz="0 -0.003 0.007"/>-->
+  		<origin rpy="0 0 ${(M_PI/2)+(reflect * (M_PI/2))}" xyz="0 ${reflect*0.003} 0.007"/>
+      <material name="black">
+        <color rgba="0.1 0.1 0.1 1"/>
+      </material>
+      </visual>
+    </link>
+    <joint name="${name}_wheelhub_joint" type="fixed">
+      <origin xyz="0 ${reflect * ((wheel_height/2) + wheel_gap + (motor_mount_width /2) )} 0" rpy="0 0 0" />
+      <parent link="${name}_motor_link"/>
+      <child link="${name}_wheelhub_link"/>
+    </joint>
+    <joint name="${name}_wheeltire_joint" type="fixed">
+      <origin xyz="0 0 0" rpy="0 0 0" />
+      <parent link="${name}_wheelhub_link"/>
+      <child link="${name}_wheeltire_link"/>
+    </joint>
+    <link name="${name}_wheelhub_link">
+      <visual>
+      <geometry>
+        <mesh filename="package://rosbee_description/meshes/wheel_hub.stl" scale="0.001 0.001 0.001"/>
+      </geometry>
+      <origin rpy="0 0 0" xyz="0 0 0"/>
+      <material name="black">
+        <color rgba="0.1 0.1 0.1 1"/>
+      </material>
+      </visual>
+    </link>
+    <link name="${name}_wheeltire_link">
+      <visual>
+      <geometry>
+        <mesh filename="package://rosbee_description/meshes/tire.stl" scale="0.001 0.001 0.001"/>
+      </geometry>
+      <origin rpy="0 0 0" xyz="0 0 0"/>
+      <material name="orange">
+        <color rgba="${240/255} ${101/255} ${26/255} 1"/>
+      </material>
+      </visual>
+    </link>
+  </xacro:macro>
+</robot>

File: rosbee_ros/rosbee_description/urdf/components/spacer.urdf.xacro (robot description, xacro)
@@ -15,5 +15,5 @@
         <cylinder radius="${spacer_diameter/2.000}" length="${spacer_height}" />
       </geometry>
-      <origin rpy="0 0 0" xyz="0 0 ${(spacer_height / 2.000) + 0.004}"/>
+      <origin rpy="0 0 0" xyz="0 0 ${(spacer_height / 2.000)}"/>
       <material name="black">
         <color rgba="0.1 0.1 0.1 1"/>

File: rosbee_ros/rosbee_description/urdf/components/top_plate.urdf.xacro (robot description, xacro)
@@ -14,5 +14,6 @@
       <visual>
       <geometry>
-        <box size="${top_plate_length} ${top_plate_width} ${top_plate_height}"/>
+        <!-- <box size="${top_plate_length} ${top_plate_width} ${top_plate_height}"/> -->
+        <mesh filename="package://rosbee_description/meshes/500085_pc_ base plate.stl" scale="0.001 0.001 0.001"/>
       </geometry>
       <origin rpy="0 0 0" xyz="0 0 0"/>

Commit message: Changes to parallax code

File: rosbee_ros/rosbee_description/robots/rosbee.urdf.xacro (robot description, xacro)
@@ -33,5 +33,5 @@
                           reflect="1"
                           offset_x="0"
-                          offset_y="0.1225"
+                          offset_y="0.127"
                           offset_z="-0.003"/>
   <xacro:motor_wheel_unit name="right"
@@ -39,5 +39,5 @@
                           reflect="-1"
                           offset_x="0"
-                          offset_y="0.1225"
+                          offset_y="0.127"
                           offset_z="-0.003"/>
   <xacro:swivel_wheel_unit name="front"

File: rosbee_ros/rosbee_description/urdf/components/motor_wheel_unit.urdf.xacro (robot description, xacro)
@@ -27,5 +27,6 @@
       <visual>
       	<geometry>
-      		<mesh filename="package://rosbee_description/meshes/500093_rvs_motormount_.stl" scale="0.02541 0.02541 0.02541"/>
+          <!--<mesh filename="package://rosbee_description/meshes/500093_rvs_motormount_.stl" scale="0.02541 0.02541 0.02541"/>-->
+          <mesh filename="package://rosbee_description/meshes/500093_RVS_motorsteun_Rosbee_mm.stl" scale="0.001 0.001 0.001"/>
       	</geometry>
       	<origin rpy="0 ${-M_PI/2} ${-reflect * M_PI/2}" xyz="0 ${reflect * motor_mount_vis_offset_y} 0"/>

Commit message: Updated Kinect Orientation

File: rosbee_ros/rosbee_description/robots/rosbee.urdf.xacro (robot description, xacro)
@@ -55,5 +55,5 @@
   <!--  kinect sensor -->
   <xacro:sensor_kinect parent="top_plate_link">
-    <origin xyz="-0.100 0.0000 0.126" rpy="0 0 -0.018516402"/>
+    <origin xyz="-0.100 0.0000 0.126" rpy="0 0 0"/>
   </xacro:sensor_kinect>
 </robot>
